Commit message: added ros2 control tag

File: robot_arm_description/urdf/arm.urdf (robot description, URDF)
Before this commit: robot robot_arm, 11 links, 10 joints
Links:
- added link tool_link
Joints:
- added joint tool_joint: type fixed, parent wrist2_link, child tool_link, origin xyz=0.0 0 0.10393 rpy=0 0 0

Commit message: updated gripper

File: robot_arm_description/urdf/arm.urdf (robot description, URDF)
Before this commit: robot robot_arm, 12 links, 11 joints
Joints:
- joint finger_joint: origin xyz=0.0 0 0 rpy=0 0 0 -> xyz=0 0 0 rpy=0 0 0
- joint gripper_joint: origin xyz=0.0 0 0.10893 rpy=0 0 0 -> xyz=0.002784 0 0.1547 rpy=0 0 0
- joint tool_joint: origin xyz=0.0 0 0.10393 rpy=0 0 0 -> xyz=0 0 -0.005 rpy=0 -3.1416 0; parent wrist2_link -> gripper_link

Commit message: removed unused servo

File: robot_arm_description/urdf/arm.urdf (robot description, URDF)
Before this commit: robot robot_arm, 12 links, 11 joints
Links:
- link wrist2_link: geometry 
Joints:
- joint gripper_joint: origin xyz=0.002784 0 0.1547 rpy=0 0 0 -> xyz=0.002784 0 0.1082 rpy=0 0 0
- joint wrist0_joint: origin xyz=0.0 0 0.175 rpy=0 0 0 -> xyz=0.0 0 0.176 rpy=0 0 0
- joint wrist2_joint: origin xyz=0.0 0 0.07005 rpy=0 0 0 -> xyz=0.0 0 0.0715 rpy=0 0 0

Commit message: added gazebo hardware interfaces

File: robot_arm_description/urdf/arm.urdf (robot description, URDF)
Before this commit: robot robot_arm, 12 links, 11 joints
Links:
- link base_link: mass None -> 0.1; geometry collision mesh filename=$(find robot_arm_description)/urdf/meshes/base_link.stl scale=0.001 0.001 0.001; visual mesh filename=$(find robot_arm_description)/urdf/meshes/base_link.stl scale=0.001 0.001 0.001
- link elbow_link: mass None -> 0.1; geometry collision mesh filename=$(find robot_arm_description)/urdf/meshes/elbow_link.stl scale=0.001 0.001 0.001; visual mesh filename=$(find robot_arm_description)/urdf/meshes/elbow_link.stl scale=0.001 0.001 0.001
- link finger_link: mass None -> 0.1; geometry collision mesh filename=$(find robot_arm_description)/urdf/meshes/finger_link.stl scale=0.001 0.001 0.001; visual mesh filename=$(find robot_arm_description)/urdf/meshes/finger_link.stl scale=0.001 0.001 0.001
- link gripper_link: mass None -> 0.1; geometry collision mesh filename=$(find robot_arm_description)/urdf/meshes/gripper_link.stl scale=0.001 0.001 0.001; visual mesh filename=$(find robot_arm_description)/urdf/meshes/gripper_link.stl scale=0.001 0.001 0.001
- link mimic_finger_link: mass None -> 0.1; geometry collision mesh filename=$(find robot_arm_description)/urdf/meshes/finger_link.stl scale=0.001 0.001 0.001; visual mesh filename=$(find robot_arm_description)/urdf/meshes/finger_link.stl scale=0.001 0.001 0.001
- link pan_link: mass None -> 0.1; geometry collision mesh filename=$(find robot_arm_description)/urdf/meshes/pan_link.stl scale=0.001 0.001 0.001; visual mesh filename=$(find robot_arm_description)/urdf/meshes/pan_link.stl scale=0.001 0.001 0.001
- link shoulder_link: mass None -> 0.1; geometry collision mesh filename=$(find robot_arm_description)/urdf/meshes/shoulder_link.stl scale=0.001 0.001 0.001; visual mesh filename=$(find robot_arm_description)/urdf/meshes/shoulder_link.stl scale=0.001 0.001 0.001
- link wrist0_link: mass None -> 0.1; geometry collision mesh filename=$(find robot_arm_description)/urdf/meshes/wrist0_link.stl scale=0.001 0.001 0.001; visual mesh filename=$(find robot_arm_description)/urdf/meshes/wrist0_link.stl scale=0.001 0.001 0.001
- link wrist1_link: mass None -> 0.1; geometry collision mesh filename=$(find robot_arm_description)/urdf/meshes/wrist1_link.stl scale=0.001 0.001 0.001; visual mesh filename=$(find robot_arm_description)/urdf/meshes/wrist1_link.stl scale=0.001 0.001 0.001
