Commit message: dynamically switch controllers between physical robot and simulated

File: robot_arm_description/urdf/arm.urdf.xacro (robot description, xacro)
@@ -1,4 +1,5 @@
 <?xml version="1.0" encoding="UTF-8"?>
-<robot name="robot_arm">
+<robot name="robot_arm" xmlns:xacro="http://ros.org/wiki/xacro">
+   <xacro:arg name="use_sim_time" default="false"/>
    <material name="black">
       <color rgba="0.15 0.15 0.15 1.0" />
@@ -9,17 +10,17 @@
          <origin rpy="0 0 0" xyz="0 0 0" />
          <geometry>
-            <mesh filename="$(find robot_arm_description)/urdf/meshes/base_link.stl" scale="0.001 0.001 0.001" />
-         </geometry>
-      </collision>
-      <visual>
-         <origin rpy="0 0 0" xyz="0 0 0" />
-         <geometry>
-            <mesh filename="$(find robot_arm_description)/urdf/meshes/base_link.stl" scale="0.001 0.001 0.001" />
-         </geometry>
-         <material name="black" />
-      </visual>
-      <inertial>
-         <mass value="0.1" />
-         <inertia ixx="0.03" iyy="0.03" izz="0.03" ixy="0.0" ixz="0.0" iyz="0.0" />
+            <mesh filename="file://$(find robot_arm_description)/urdf/meshes/base_link.stl" scale="0.001 0.001 0.001" />
+         </geometry>
+      </collision>
+      <visual>
+         <origin rpy="0 0 0" xyz="0 0 0" />
+         <geometry>
+            <mesh filename="file://$(find robot_arm_description)/urdf/meshes/base_link.stl" scale="0.001 0.001 0.001" />
+         </geometry>
+         <material name="black" />
+      </visual>
+      <inertial>
+         <mass value="50" />
+         <inertia ixx="0.1" iyy="0.1" izz="0.1" ixy="0.0" ixz="0.0" iyz="0.0" />
       </inertial>
    </link>
@@ -33,11 +34,11 @@
          <origin rpy="0 0 0" xyz="0 0 0" />
          <geometry>
-            <mesh filename="$(find robot_arm_description)/urdf/meshes/pan_link.stl" scale="0.001 0.001 0.001" />
-         </geometry>
-      </collision>
-      <visual>
-         <origin rpy="0 0 0" xyz="0 0 0" />
-         <geometry>
-            <mesh filename="$(find robot_arm_description)/urdf/meshes/pan_link.stl" scale="0.001 0.001 0.001" />
+            <mesh filename="file://$(find robot_arm_description)/urdf/meshes/pan_link.stl" scale="0.001 0.001 0.001" />
+         </geometry>
+      </collision>
+      <visual>
+         <origin rpy="0 0 0" xyz="0 0 0" />
+         <geometry>
+            <mesh filename="file://$(find robot_arm_description)/urdf/meshes/pan_link.stl" scale="0.001 0.001 0.001" />
          </geometry>
          <material name="black" />
@@ -59,11 +60,11 @@
          <origin rpy="0 0 0" xyz="0 0 0" />
          <geometry>
-            <mesh filename="$(find robot_arm_description)/urdf/meshes/shoulder_link.stl" scale="0.001 0.001 0.001" />
-         </geometry>
-      </collision>
-      <visual>
-         <origin rpy="0 0 0" xyz="0 0 0" />
-         <geometry>
-            <mesh filename="$(find robot_arm_description)/urdf/meshes/shoulder_link.stl" scale="0.001 0.001 0.001" />
+            <mesh filename="file://$(find robot_arm_description)/urdf/meshes/shoulder_link.stl" scale="0.001 0.001 0.001" />
+         </geometry>
+      </collision>
+      <visual>
+         <origin rpy="0 0 0" xyz="0 0 0" />
+         <geometry>
+            <mesh filename="file://$(find robot_arm_description)/urdf/meshes/shoulder_link.stl" scale="0.001 0.001 0.001" />
          </geometry>
          <material name="black" />
@@ -85,11 +86,11 @@
          <origin rpy="0 0 0" xyz="0 0 0" />
          <geometry>
-            <mesh filename="$(find robot_arm_description)/urdf/meshes/elbow_link.stl" scale="0.001 0.001 0.001" />
-         </geometry>
-      </collision>
-      <visual>
-         <origin rpy="0 0 0" xyz="0 0 0" />
-         <geometry>
-            <mesh filename="$(find robot_arm_description)/urdf/meshes/elbow_link.stl" scale="0.001 0.001 0.001" />
+            <mesh filename="file://$(find robot_arm_description)/urdf/meshes/elbow_link.stl" scale="0.001 0.001 0.001" />
+         </geometry>
+      </collision>
+      <visual>
+         <origin rpy="0 0 0" xyz="0 0 0" />
+         <geometry>
+            <mesh filename="file://$(find robot_arm_description)/urdf/meshes/elbow_link.stl" scale="0.001 0.001 0.001" />
          </geometry>
          <material name="black" />
@@ -111,11 +112,11 @@
          <origin rpy="0 0 0" xyz="0 0 0" />
          <geometry>
-            <mesh filename="$(find robot_arm_description)/urdf/meshes/wrist0_link.stl" scale="0.001 0.001 0.001" />
-         </geometry>
-      </collision>
-      <visual>
-         <origin rpy="0 0 0" xyz="0 0 0" />
-         <geometry>
-            <mesh filename="$(find robot_arm_description)/urdf/meshes/wrist0_link.stl" scale="0.001 0.001 0.001" />
+            <mesh filename="file://$(find robot_arm_description)/urdf/meshes/wrist0_link.stl" scale="0.001 0.001 0.001" />
+         </geometry>
+      </collision>
+      <visual>
+         <origin rpy="0 0 0" xyz="0 0 0" />
+         <geometry>
+            <mesh filename="file://$(find robot_arm_description)/urdf/meshes/wrist0_link.stl" scale="0.001 0.001 0.001" />
          </geometry>
          <material name="black" />
@@ -137,11 +138,11 @@
          <origin rpy="0 0 0" xyz="0 0 0" />
          <geometry>
-            <mesh filename="$(find robot_arm_description)/urdf/meshes/wrist1_link.stl" scale="0.001 0.001 0.001" />
-         </geometry>
-      </collision>
-      <visual>
-         <origin rpy="0 0 0" xyz="0 0 0" />
-         <geometry>
-            <mesh filename="$(find robot_arm_description)/urdf/meshes/wrist1_link.stl" scale="0.001 0.001 0.001" />
+            <mesh filename="file://$(find robot_arm_description)/urdf/meshes/wrist1_link.stl" scale="0.001 0.001 0.001" />
+         </geometry>
+      </collision>
+      <visual>
+         <origin rpy="0 0 0" xyz="0 0 0" />
+         <geometry>
+            <mesh filename="file://$(find robot_arm_description)/urdf/meshes/wrist1_link.stl" scale="0.001 0.001 0.001" />
          </geometry>
          <material name="black" />
@@ -171,11 +172,11 @@
          <origin rpy="0 0 0" xyz="0 0 0" />
          <geometry>
-            <mesh filename="$(find robot_arm_description)/urdf/meshes/gripper_link.stl" scale="0.001 0.001 0.001" />
-         </geometry>
-      </collision>
-      <visual>
-         <origin rpy="0 0 0" xyz="0 0 0" />
-         <geometry>
-            <mesh filename="$(find robot_arm_description)/urdf/meshes/gripper_link.stl" scale="0.001 0.001 0.001" />
+            <mesh filename="file://$(find robot_arm_description)/urdf/meshes/gripper_link.stl" scale="0.001 0.001 0.001" />
+         </geometry>
+      </collision>
+      <visual>
+         <origin rpy="0 0 0" xyz="0 0 0" />
+         <geometry>
+            <mesh filename="file://$(find robot_arm_description)/urdf/meshes/gripper_link.stl" scale="0.001 0.001 0.001" />
          </geometry>
          <material name="black" />
@@ -195,11 +196,11 @@
          <origin rpy="0 0 0" xyz="0 0 0" />
          <geometry>
-            <mesh filename="$(find robot_arm_description)/urdf/meshes/finger_link.stl" scale="0.001 0.001 0.001" />
-         </geometry>
-      </collision>
-      <visual>
-         <origin rpy="0 0 0" xyz="0 0 0" />
-         <geometry>
-            <mesh filename="$(find robot_arm_description)/urdf/meshes/finger_link.stl" scale="0.001 0.001 0.001" />
+            <mesh filename="file://$(find robot_arm_description)/urdf/meshes/finger_link.stl" scale="0.001 0.001 0.001" />
+         </geometry>
+      </collision>
+      <visual>
+         <origin rpy="0 0 0" xyz="0 0 0" />
+         <geometry>
+            <mesh filename="file://$(find robot_arm_description)/urdf/meshes/finger_link.stl" scale="0.001 0.001 0.001" />
          </geometry>
          <material name="black" />
@@ -221,5 +222,5 @@
          <origin rpy="0 0 3.1416" xyz="0 0 0" />
          <geometry>
-            <mesh filename="$(find robot_arm_description)/urdf/meshes/finger_link.stl" scale="0.001 0.001 0.001" />
+            <mesh filename="file://$(find robot_arm_description)/urdf/meshes/finger_link.stl" scale="0.001 0.001 0.001" />
          </geometry>
       </collision>
@@ -227,5 +228,5 @@
          <origin rpy="0 0 3.1416" xyz="0 0 0" />
          <geometry>
-            <mesh filename="$(find robot_arm_description)/urdf/meshes/finger_link.stl" scale="0.001 0.001 0.001" />
+            <mesh filename="file://$(find robot_arm_description)/urdf/meshes/finger_link.stl" scale="0.001 0.001 0.001" />
          </geometry>
          <material name="black" />
@@ -239,8 +240,8 @@
       <axis xyz="0 1 0" />
       <mimic joint="finger_joint" multiplier="-1" />
-      <limit lower="-0.026" upper="0" effort="1.0" velocity="0" />
-      <parent link="gripper_link" />
-      <child link="mimic_finger_link" />
-      <origin rpy="0 0 0" xyz="0.0 0 0" />
+      <limit lower="0.026" upper="0" effort="1.0" velocity="0" />
+      <parent link="gripper_link"/>
+      <child link="mimic_finger_link"/>
+      <origin rpy="0 0 0" xyz="0.0 0 0"/>
    </joint>
    <link name="tool_link" />
@@ -251,11 +252,21 @@
    </joint>
    <ros2_control name="robot_arm" type="system">
-      <hardware>
-         <plugin>gazebo_ros2_control/GazeboSystem</plugin>
-      </hardware>
+      <xacro:if value="$(arg use_sim_time)">
+         <hardware>
+            <plugin>gazebo_ros2_control/GazeboSystem</plugin>
+         </hardware>
+      </xacro:if>
+      <xacro:unless value="$(arg use_sim_time)">
+         <hardware>
+            <plugin>fake_components/GenericSystem</plugin>
+         </hardware>
+      </xacro:unless>
       <joint name="mimic_finger_joint">
          <param name="mimic">finger_joint</param>
          <param name="multiplier">-1</param>
-         <command_interface name="position" />
+         <command_interface name="position">
+            <param name="min">0</param>
+            <param name="max">0.026</param>
+         </command_interface>
          <state_interface name="position" />
          <state_interface name="velocity" />
@@ -264,6 +275,6 @@
       <joint name="pan_joint">
          <command_interface name="position">
-            <param name="min">-1000</param>
-            <param name="max">1000</param>
+            <param name="min">-3.1416</param>
+            <param name="max">3.1416</param>
          </command_interface>
          <state_interface name="position" />
@@ -273,6 +284,6 @@
       <joint name="shoulder_joint">
          <command_interface name="position">
-            <param name="min">-1000</param>
-            <param name="max">1000</param>
+            <param name="min">-3.1416</param>
+            <param name="max">3.1416</param>
          </command_interface>
          <state_interface name="position" />
@@ -282,6 +293,6 @@
       <joint name="elbow_joint">
          <command_interface name="position">
-            <param name="min">-1000</param>
-            <param name="max">1000</param>
+            <param name="min">-3.1416</param>
+            <param name="max">3.1416</param>
          </command_interface>
          <state_interface name="position" />
@@ -291,6 +302,6 @@
       <joint name="wrist0_joint">
          <command_interface name="position">
-            <param name="min">-1000</param>
-            <param name="max">1000</param>
+            <param name="min">-3.1416</param>
+            <param name="max">3.1416</param>
          </command_interface>
          <state_interface name="position" />
@@ -300,6 +311,6 @@
       <joint name="wrist1_joint">
          <command_interface name="position">
-            <param name="min">-1000</param>
-            <param name="max">1000</param>
+            <param name="min">-3.1416</param>
+            <param name="max">3.1416</param>
          </command_interface>
          <state_interface name="position" />
@@ -309,6 +320,6 @@
       <joint name="wrist2_joint">
          <command_interface name="position">
-            <param name="min">-1000</param>
-            <param name="max">1000</param>
+            <param name="min">-3.1416</param>
+            <param name="max">3.1416</param>
          </command_interface>
          <state_interface name="position" />
@@ -318,6 +329,6 @@
       <joint name="finger_joint">
          <command_interface name="position">
-            <param name="min">-1000</param>
-            <param name="max">1000</param>
+            <param name="min">-3.1416</param>
+            <param name="max">3.1416</param>
          </command_interface>
          <state_interface name="position" />
@@ -327,5 +338,5 @@
    </ros2_control>
    <gazebo>
-      <plugin filename="libgazebo_ros2_control.so" name="gazebo_ros2_control">
+      <plugin filename="libgazebo_ros2_control.so" name="gazebo_ros2_control_urdf">
          <robot_param>robot_description</robot_param>
          <robot_param_node>robot_state_publisher</robot_param_node>

Commit message: sync up color

File: robot_arm_description/urdf/arm.urdf.xacro (robot description, xacro)
@@ -1,5 +1,5 @@
 <?xml version="1.0" encoding="UTF-8"?>
-<robot name="robot_arm" xmlns:xacro="http://ros.org/wiki/xacro">
-   <xacro:arg name="use_sim_time" default="false"/>
+<robot xmlns:xacro="http://ros.org/wiki/xacro" name="robot_arm">
+   <xacro:arg name="use_sim_time" default="false" />
    <material name="black">
       <color rgba="0.15 0.15 0.15 1.0" />
@@ -25,4 +25,7 @@
       </inertial>
    </link>
+   <gazebo reference="base_link">
+      <material>Gazebo/FlatBlack</material>
+   </gazebo>
    <joint name="base_to_mount" type="fixed">
       <parent link="base_mount" />
@@ -49,4 +52,7 @@
       </inertial>
    </link>
+   <gazebo reference="pan_link">
+      <material>Gazebo/FlatBlack</material>
+   </gazebo>
    <joint name="pan_joint" type="revolute">
       <axis xyz="0 0 1" />
@@ -75,4 +81,7 @@
       </inertial>
    </link>
+   <gazebo reference="shoulder_link">
+      <material>Gazebo/FlatBlack</material>
+   </gazebo>
    <joint name="shoulder_joint" type="revolute">
       <axis xyz="0 1 0" />
@@ -101,4 +110,7 @@
       </inertial>
    </link>
+   <gazebo reference="elbow_link">
+      <material>Gazebo/FlatBlack</material>
+   </gazebo>
    <joint name="elbow_joint" type="revolute">
       <axis xyz="0 1 0" />
@@ -127,4 +139,7 @@
       </inertial>
    </link>
+   <gazebo reference="wrist0_link">
+      <material>Gazebo/FlatBlack</material>
+   </gazebo>
    <joint name="wrist0_joint" type="revolute">
       <axis xyz="0 0 1" />
@@ -134,4 +149,7 @@
       <origin rpy="0 0 0" xyz="0.0 0 0.176" />
    </joint>
+   <gazebo reference="wrist1_link">
+      <material>Gazebo/FlatBlack</material>
+   </gazebo>
    <link name="wrist1_link">
       <collision>
@@ -153,4 +171,7 @@
       </inertial>
    </link>
+   <gazebo reference="wrist1_link">
+      <material>Gazebo/FlatBlack</material>
+   </gazebo>
    <joint name="wrist1_joint" type="revolute">
       <axis xyz="0 1 0" />
@@ -187,4 +208,7 @@
       </inertial>
    </link>
+   <gazebo reference="gripper_link">
+      <material>Gazebo/FlatBlack</material>
+   </gazebo>
    <joint name="gripper_joint" type="fixed">
       <parent link="wrist2_link" />
@@ -211,4 +235,7 @@
       </inertial>
    </link>
+   <gazebo reference="finger_link">
+      <material>Gazebo/FlatBlack</material>
+   </gazebo>
    <joint name="finger_joint" type="prismatic">
       <axis xyz="0 1 0" />
@@ -237,11 +264,14 @@
       </inertial>
    </link>
+   <gazebo reference="mimic_finger_link">
+      <material>Gazebo/FlatBlack</material>
+   </gazebo>
    <joint name="mimic_finger_joint" type="prismatic">
       <axis xyz="0 1 0" />
       <mimic joint="finger_joint" multiplier="-1" />
       <limit lower="0.026" upper="0" effort="1.0" velocity="0" />
-      <parent link="gripper_link"/>
-      <child link="mimic_finger_link"/>
-      <origin rpy="0 0 0" xyz="0.0 0 0"/>
+      <parent link="gripper_link" />
+      <child link="mimic_finger_link" />
+      <origin rpy="0 0 0" xyz="0.0 0 0" />
    </joint>
    <link name="tool_link" />

Commit message: renamed base_link to base_link

File: robot_arm_description/urdf/arm.urdf.xacro (robot description, xacro)
@@ -6,15 +6,15 @@
    </material>
    <link name="base_mount" />
-   <link name="base_link">
-      <collision>
-         <origin rpy="0 0 0" xyz="0 0 0" />
-         <geometry>
-            <mesh filename="file://$(find robot_arm_description)/urdf/meshes/base_link.stl" scale="0.001 0.001 0.001" />
-         </geometry>
-      </collision>
-      <visual>
-         <origin rpy="0 0 0" xyz="0 0 0" />
-         <geometry>
-            <mesh filename="file://$(find robot_arm_description)/urdf/meshes/base_link.stl" scale="0.001 0.001 0.001" />
+   <link name="box_link">
+      <collision>
+         <origin rpy="0 0 0" xyz="0 0 0" />
+         <geometry>
+            <mesh filename="file://$(find robot_arm_description)/urdf/meshes/box_link.stl" scale="0.001 0.001 0.001" />
+         </geometry>
+      </collision>
+      <visual>
+         <origin rpy="0 0 0" xyz="0 0 0" />
+         <geometry>
+            <mesh filename="file://$(find robot_arm_description)/urdf/meshes/box_link.stl" scale="0.001 0.001 0.001" />
          </geometry>
          <material name="black" />
@@ -25,10 +25,10 @@
       </inertial>
    </link>
-   <gazebo reference="base_link">
+   <gazebo reference="box_link">
       <material>Gazebo/FlatBlack</material>
    </gazebo>
    <joint name="base_to_mount" type="fixed">
       <parent link="base_mount" />
-      <child link="base_link" />
+      <child link="box_link" />
       <origin rpy="0 0 0" xyz="0 0 0.0575" />
    </joint>
@@ -58,5 +58,5 @@
       <axis xyz="0 0 1" />
       <limit effort="25" lower="-3.14159265359" upper="3.14159265359" velocity="1.5" />
-      <parent link="base_link" />
+      <parent link="box_link" />
       <child link="pan_link" />
       <origin rpy="0 0 0" xyz="-0.012 0 0.002" />
