Commit message: make URDF importable from another URDF

File: robot_arm_description/urdf/arm.urdf.xacro (robot description, xacro)
@@ -2,375 +2,24 @@
 <robot xmlns:xacro="http://ros.org/wiki/xacro" name="robot_arm">
    <xacro:arg name="use_sim_time" default="false" />
-   <material name="black">
-      <color rgba="0.15 0.15 0.15 1.0" />
-   </material>
-   <link name="base_mount" />
-   <link name="box_link">
+   <xacro:include filename="$(find robot_arm_description)/urdf/arm_mech.urdf.xacro" />
+  <link name="base_mount">
       <collision>
-         <origin rpy="0 0 0" xyz="0 0 0" />
-         <geometry>
-            <mesh filename="file://$(find robot_arm_description)/urdf/meshes/box_link.stl" scale="0.001 0.001 0.001" />
-         </geometry>
+        <origin rpy="0 0 0" xyz="0 0 0" />
+        <geometry>
+            <mesh filename="file://$(find robot_arm_description)/urdf/meshes/base_mount.stl" scale="0.001 0.001 0.001" />
+        </geometry>
       </collision>
       <visual>
-         <origin rpy="0 0 0" xyz="0 0 0" />
-         <geometry>
-            <mesh filename="file://$(find robot_arm_description)/urdf/meshes/box_link.stl" scale="0.001 0.001 0.001" />
-         </geometry>
-         <material name="black" />
+        <origin rpy="0 0 0" xyz="0 0 0" />
+        <geometry>
+            <mesh filename="file://$(find robot_arm_description)/urdf/meshes/base_mount.stl" scale="0.001 0.001 0.001" />
+        </geometry>
+        <material name="black" />
       </visual>
       <inertial>
-         <mass value="50" />
-         <inertia ixx="0.1" iyy="0.1" izz="0.1" ixy="0.0" ixz="0.0" iyz="0.0" />
+        <mass value="50" />
+        <inertia ixx="0.1" iyy="0.1" izz="0.1" ixy="0.0" ixz="0.0" iyz="0.0" />
       </inertial>
-   </link>
-   <gazebo reference="box_link">
-      <material>Gazebo/FlatBlack</material>
-   </gazebo>
-   <joint name="base_to_mount" type="fixed">
-      <parent link="base_mount" />
-      <child link="box_link" />
-      <origin rpy="0 0 0" xyz="0 0 0.0575" />
-   </joint>
-   <link name="pan_link">
-      <collision>
-         <origin rpy="0 0 0" xyz="0 0 0" />
-         <geometry>
-            <mesh filename="file://$(find robot_arm_description)/urdf/meshes/pan_link.stl" scale="0.001 0.001 0.001" />
-         </geometry>
-      </collision>
-      <visual>
-         <origin rpy="0 0 0" xyz="0 0 0" />
-         <geometry>
-            <mesh filename="file://$(find robot_arm_description)/urdf/meshes/pan_link.stl" scale="0.001 0.001 0.001" />
-         </geometry>
-         <material name="black" />
-      </visual>
-      <inertial>
-         <mass value="0.1" />
-         <inertia ixx="0.03" iyy="0.03" izz="0.03" ixy="0.0" ixz="0.0" iyz="0.0" />
-      </inertial>
-   </link>
-   <gazebo reference="pan_link">
-      <material>Gazebo/FlatBlack</material>
-   </gazebo>
-   <joint name="pan_joint" type="revolute">
-      <axis xyz="0 0 1" />
-      <limit effort="25" lower="-3.14159265359" upper="3.14159265359" velocity="1.5" />
-      <parent link="box_link" />
-      <child link="pan_link" />
-      <origin rpy="0 0 0" xyz="-0.012 0 0.002" />
-   </joint>
-   <link name="shoulder_link">
-      <collision>
-         <origin rpy="0 0 0" xyz="0 0 0" />
-         <geometry>
-            <mesh filename="file://$(find robot_arm_description)/urdf/meshes/shoulder_link.stl" scale="0.001 0.001 0.001" />
-         </geometry>
-      </collision>
-      <visual>
-         <origin rpy="0 0 0" xyz="0 0 0" />
-         <geometry>
-            <mesh filename="file://$(find robot_arm_description)/urdf/meshes/shoulder_link.stl" scale="0.001 0.001 0.001" />
-         </geometry>
-         <material name="black" />
-      </visual>
-      <inertial>
-         <mass value="0.1" />
-         <inertia ixx="0.03" iyy="0.03" izz="0.03" ixy="0.0" ixz="0.0" iyz="0.0" />
-      </inertial>
-   </link>
-   <gazebo reference="shoulder_link">
-      <material>Gazebo/FlatBlack</material>
-   </gazebo>
-   <joint name="shoulder_joint" type="revolute">
-      <axis xyz="0 1 0" />
-      <limit effort="25" lower="-1.8515" upper="2.1015" velocity="1.5" />
-      <parent link="pan_link" />
-      <child link="shoulder_link" />
-      <origin rpy="0 0 0" xyz="0 0 0.053" />
-   </joint>
-   <link name="elbow_link">
-      <collision>
-         <origin rpy="0 0 0" xyz="0 0 0" />
-         <geometry>
-            <mesh filename="file://$(find robot_arm_description)/urdf/meshes/elbow_link.stl" scale="0.001 0.001 0.001" />
-         </geometry>
-      </collision>
-      <visual>
-         <origin rpy="0 0 0" xyz="0 0 0" />
-         <geometry>
-            <mesh filename="file://$(find robot_arm_description)/urdf/meshes/elbow_link.stl" scale="0.001 0.001 0.001" />
-         </geometry>
-         <material name="black" />
-      </visual>
-      <inertial>
-         <mass value="0.1" />
-         <inertia ixx="0.03" iyy="0.03" izz="0.03" ixy="0.0" ixz="0.0" iyz="0.0" />
-      </inertial>
-   </link>
-   <gazebo reference="elbow_link">
-      <material>Gazebo/FlatBlack</material>
-   </gazebo>
-   <joint name="elbow_joint" type="revolute">
-      <axis xyz="0 1 0" />
-      <limit effort="25" lower="-0.4" upper="3.0" velocity="1.5" />
-      <parent link="shoulder_link" />
-      <child link="elbow_link" />
-      <origin rpy="0 0 0" xyz="0.03 0 0.2205" />
-   </joint>
-   <link name="wrist0_link">
-      <collision>
-         <origin rpy="0 0 0" xyz="0 0 0" />
-         <geometry>
-            <mesh filename="file://$(find robot_arm_description)/urdf/meshes/wrist0_link.stl" scale="0.001 0.001 0.001" />
-         </geometry>
-      </collision>
-      <visual>
-         <origin rpy="0 0 0" xyz="0 0 0" />
-         <geometry>
-            <mesh filename="file://$(find robot_arm_description)/urdf/meshes/wrist0_link.stl" scale="0.001 0.001 0.001" />
-         </geometry>
-         <material name="black" />
-      </visual>
-      <inertial>
-         <mass value="0.1" />
-         <inertia ixx="0.03" iyy="0.03" izz="0.03" ixy="0.0" ixz="0.0" iyz="0.0" />
-      </inertial>
-   </link>
-   <gazebo reference="wrist0_link">
-      <material>Gazebo/FlatBlack</material>
-   </gazebo>
-   <joint name="wrist0_joint" type="revolute">
-      <axis xyz="0 0 1" />
-      <limit effort="25" lower="-3.14159265359" upper="3.14159265359" velocity="1.5" />
-      <parent link="elbow_link" />
-      <child link="wrist0_link" />
-      <origin rpy="0 0 0" xyz="0.0 0 0.176" />
-   </joint>
-   <gazebo reference="wrist1_link">
-      <material>Gazebo/FlatBlack</material>
-   </gazebo>
-   <link name="wrist1_link">
-      <collision>
-         <origin rpy="0 0 0" xyz="0 0 0" />
-         <geometry>
-            <mesh filename="file://$(find robot_arm_description)/urdf/meshes/wrist1_link.stl" scale="0.001 0.001 0.001" />
-         </geometry>
-      </collision>
-      <visual>
-         <origin rpy="0 0 0" xyz="0 0 0" />
-         <geometry>
-            <mesh filename="file://$(find robot_arm_description)/urdf/meshes/wrist1_link.stl" scale="0.001 0.001 0.001" />
-         </geometry>
-         <material name="black" />
-      </visual>
-      <inertial>
-         <mass value="0.1" />
-         <inertia ixx="0.03" iyy="0.03" izz="0.03" ixy="0.0" ixz="0.0" iyz="0.0" />
-      </inertial>
-   </link>
-   <gazebo reference="wrist1_link">
-      <material>Gazebo/FlatBlack</material>
-   </gazebo>
-   <joint name="wrist1_joint" type="revolute">
-      <axis xyz="0 1 0" />
-      <limit effort="25" lower="-1.8" upper="2.0" velocity="1.5" />
-      <parent link="wrist0_link" />
-      <child link="wrist1_link" />
-      <origin rpy="0 0 0" xyz="0.0 0 0.0435" />
-   </joint>
-   <link name="wrist2_link" />
-   <joint name="wrist2_joint" type="revolute">
-      <axis xyz="0 0 1" />
-      <limit effort="25" lower="-3.14159265359" upper="3.14159265359" velocity="1.5" />
-      <parent link="wrist1_link" />
-      <child link="wrist2_link" />
-      <origin rpy="0 0 0" xyz="0.0 0 0.0715" />
-   </joint>
-   <link name="gripper_link">
-      <collision>
-         <origin rpy="0 0 0" xyz="0 0 0" />
-         <geometry>
-            <mesh filename="file://$(find robot_arm_description)/urdf/meshes/gripper_link.stl" scale="0.001 0.001 0.001" />
-         </geometry>
-      </collision>
-      <visual>
-         <origin rpy="0 0 0" xyz="0 0 0" />
-         <geometry>
-            <mesh filename="file://$(find robot_arm_description)/urdf/meshes/gripper_link.stl" scale="0.001 0.001 0.001" />
-         </geometry>
-         <material name="black" />
-      </visual>
-      <inertial>
-         <mass value="0.1" />
-         <inertia ixx="0.03" iyy="0.03" izz="0.03" ixy="0.0" ixz="0.0" iyz="0.0" />
-      </inertial>
-   </link>
-   <gazebo reference="gripper_link">
-      <material>Gazebo/FlatBlack</material>
-   </gazebo>
-   <joint name="gripper_joint" type="fixed">
-      <parent link="wrist2_link" />
-      <child link="gripper_link" />
-      <origin rpy="0 0 0" xyz="0.002784 0 0.1082" />
-   </joint>
-   <link name="finger_link">
-      <collision>
-         <origin rpy="0 0 0" xyz="0 0 0" />
-         <geometry>
-            <mesh filename="file://$(find robot_arm_description)/urdf/meshes/finger_link.stl" scale="0.001 0.001 0.001" />
-         </geometry>
-      </collision>
-      <visual>
-         <origin rpy="0 0 0" xyz="0 0 0" />
-         <geometry>
-            <mesh filename="file://$(find robot_arm_description)/urdf/meshes/finger_link.stl" scale="0.001 0.001 0.001" />
-         </geometry>
-         <material name="black" />
-      </visual>
-      <inertial>
-         <mass value="0.1" />
-         <inertia ixx="0.03" iyy="0.03" izz="0.03" ixy="0.0" ixz="0.0" iyz="0.0" />
-      </inertial>
-   </link>
-   <gazebo reference="finger_link">
-      <material>Gazebo/FlatBlack</material>
-   </gazebo>
-   <joint name="finger_joint" type="prismatic">
-      <axis xyz="0 1 0" />
-      <limit lower="0" upper="0.026" effort="1.0" velocity="0" />
-      <parent link="gripper_link" />
-      <child link="finger_link" />
-      <origin rpy="0 0 0" xyz="0 0 0" />
-   </joint>
-   <link name="mimic_finger_link">
-      <collision>
-         <origin rpy="0 0 3.1416" xyz="0 0 0" />
-         <geometry>
-            <mesh filename="file://$(find robot_arm_description)/urdf/meshes/finger_link.stl" scale="0.001 0.001 0.001" />
-         </geometry>
-      </collision>
-      <visual>
-         <origin rpy="0 0 3.1416" xyz="0 0 0" />
-         <geometry>
-            <mesh filename="file://$(find robot_arm_description)/urdf/meshes/finger_link.stl" scale="0.001 0.001 0.001" />
-         </geometry>
-         <material name="black" />
-      </visual>
-      <inertial>
-         <mass value="0.1" />
-         <inertia ixx="0.03" iyy="0.03" izz="0.03" ixy="0.0" ixz="0.0" iyz="0.0" />
-      </inertial>
-   </link>
-   <gazebo reference="mimic_finger_link">
-      <material>Gazebo/FlatBlack</material>
-   </gazebo>
-   <joint name="mimic_finger_joint" type="prismatic">
-      <axis xyz="0 1 0" />
-      <mimic joint="finger_joint" multiplier="-1" />
-      <limit lower="0.026" upper="0" effort="1.0" velocity="0" />
-      <parent link="gripper_link" />
-      <child link="mimic_finger_link" />
-      <origin rpy="0 0 0" xyz="0.0 0 0" />
-   </joint>
-   <link name="tool_link" />
-   <joint name="tool_joint" type="fixed">
-      <parent link="gripper_link" />
-      <child link="tool_link" />
-      <origin rpy="0 -3.1416 0" xyz="0 0 -0.005" />
-   </joint>
-   <ros2_control name="robot_arm" type="system">
-      <xacro:if value="$(arg use_sim_time)">
-         <hardware>
-            <plugin>gazebo_ros2_control/GazeboSystem</plugin>
-         </hardware>
-      </xacro:if>
-      <xacro:unless value="$(arg use_sim_time)">
-         <hardware>
-            <plugin>fake_components/GenericSystem</plugin>
-         </hardware>
-      </xacro:unless>
-      <joint name="mimic_finger_joint">
-         <param name="mimic">finger_joint</param>
-         <param name="multiplier">-1</param>
-         <command_interface name="position">
-            <param name="min">0</param>
-            <param name="max">0.026</param>
-         </command_interface>
-         <state_interface name="position" />
-         <state_interface name="velocity" />
-         <state_interface name="effort" />
-      </joint>
-      <joint name="pan_joint">
-         <command_interface name="position">
-            <param name="min">-3.1416</param>
-            <param name="max">3.1416</param>
-         </command_interface>
-         <state_interface name="position" />
-         <state_interface name="velocity" />
-         <state_interface name="effort" />
-      </joint>
-      <joint name="shoulder_joint">
-         <command_interface name="position">
-            <param name="min">-3.1416</param>
-            <param name="max">3.1416</param>
-         </command_interface>
-         <state_interface name="position" />
-         <state_interface name="velocity" />
-         <state_interface name="effort" />
-      </joint>
-      <joint name="elbow_joint">
-         <command_interface name="position">
-            <param name="min">-3.1416</param>
-            <param name="max">3.1416</param>
-         </command_interface>
-         <state_interface name="position" />
-         <state_interface name="velocity" />
-         <state_interface name="effort" />
-      </joint>
-      <joint name="wrist0_joint">
-         <command_interface name="position">
-            <param name="min">-3.1416</param>
-            <param name="max">3.1416</param>
-         </command_interface>
-         <state_interface name="position" />
-         <state_interface name="velocity" />
-         <state_interface name="effort" />
-      </joint>
-      <joint name="wrist1_joint">
-         <command_interface name="position">
-            <param name="min">-3.1416</param>
-            <param name="max">3.1416</param>
-         </command_interface>
-         <state_interface name="position" />
-         <state_interface name="velocity" />
-         <state_interface name="effort" />
-      </joint>
-      <joint name="wrist2_joint">
-         <command_interface name="position">
-            <param name="min">-3.1416</param>
-            <param name="max">3.1416</param>
-         </command_interface>
-         <state_interface name="position" />
-         <state_interface name="velocity" />
-         <state_interface name="effort" />
-      </joint>
-      <joint name="finger_joint">
-         <command_interface name="position">
-            <param name="min">-3.1416</param>
-            <param name="max">3.1416</param>
-         </command_interface>
-         <state_interface name="position" />
-         <state_interface name="velocity" />
-         <state_interface name="effort" />
-      </joint>
-   </ros2_control>
-   <gazebo>
-      <plugin filename="libgazebo_ros2_control.so" name="gazebo_ros2_control_urdf">
-         <robot_param>robot_description</robot_param>
-         <robot_param_node>robot_state_publisher</robot_param_node>
-         <parameters>$(find robot_arm_description)/config/controller.yaml</parameters>
-      </plugin>
-   </gazebo>
+  </link>
+  <xacro:arm_mech parent="base_mount" use_sim_time="$(arg use_sim_time)" />
 </robot>
