Commit message: fixed formatting

File: robot_arm_description/urdf/arm.urdf.xacro (robot description, xacro)
@@ -3,23 +3,26 @@
    <xacro:arg name="use_sim_time" default="false" />
    <xacro:include filename="$(find robot_arm_description)/urdf/arm_mech.urdf.xacro" />
-  <link name="base_mount">
+   <material name="black">
+      <color rgba="0.15 0.15 0.15 1.0" />
+   </material>
+   <link name="base_mount">
       <collision>
-        <origin rpy="0 0 0" xyz="0 0 0" />
-        <geometry>
+         <origin rpy="0 0 0" xyz="0 0 0" />
+         <geometry>
             <mesh filename="file://$(find robot_arm_description)/urdf/meshes/base_mount.stl" scale="0.001 0.001 0.001" />
-        </geometry>
+         </geometry>
       </collision>
       <visual>
-        <origin rpy="0 0 0" xyz="0 0 0" />
-        <geometry>
+         <origin rpy="0 0 0" xyz="0 0 0" />
+         <geometry>
             <mesh filename="file://$(find robot_arm_description)/urdf/meshes/base_mount.stl" scale="0.001 0.001 0.001" />
-        </geometry>
-        <material name="black" />
+         </geometry>
+         <material name="black" />
       </visual>
       <inertial>
-        <mass value="50" />
-        <inertia ixx="0.1" iyy="0.1" izz="0.1" ixy="0.0" ixz="0.0" iyz="0.0" />
+         <mass value="50" />
+         <inertia ixx="0.1" iyy="0.1" izz="0.1" ixy="0.0" ixz="0.0" iyz="0.0" />
       </inertial>
-  </link>
-  <xacro:arm_mech parent="base_mount" use_sim_time="$(arg use_sim_time)" />
+   </link>
+   <xacro:arm_mech parent="base_mount" use_sim_time="$(arg use_sim_time)" />
 </robot>

File: robot_arm_description/urdf/arm_mech.urdf.xacro (robot description, xacro)
@@ -1,376 +1,373 @@
 <?xml version="1.0" encoding="UTF-8"?>
 <robot xmlns:xacro="http://ros.org/wiki/xacro" name="robot_arm">
-   <xacro:macro name="arm_mech" params="use_sim_time parent">
-      <material name="black">
-         <color rgba="0.15 0.15 0.15 1.0" />
-      </material>
-      <link name="box_link">
-         <collision>
+    <xacro:macro name="arm_mech" params="use_sim_time parent">
+        <link name="box_link">
+            <collision>
+                <origin rpy="0 0 0" xyz="0 0 0" />
+                <geometry>
+                    <mesh filename="file://$(find robot_arm_description)/urdf/meshes/box_link.stl" scale="0.001 0.001 0.001" />
+                </geometry>
+            </collision>
+            <visual>
+                <origin rpy="0 0 0" xyz="0 0 0" />
+                <geometry>
+                    <mesh filename="file://$(find robot_arm_description)/urdf/meshes/box_link.stl" scale="0.001 0.001 0.001" />
+                </geometry>
+                <material name="black" />
+            </visual>
+            <inertial>
+                <mass value="0.1" />
+                <inertia ixx="0.1" iyy="0.1" izz="0.1" ixy="0.0" ixz="0.0" iyz="0.0" />
+            </inertial>
+        </link>
+        <gazebo reference="box_link">
+            <material>Gazebo/FlatBlack</material>
+        </gazebo>
+        <joint name="base_to_mount" type="fixed">
+            <parent link="${parent}" />
+            <child link="box_link" />
+            <origin rpy="0 0 0" xyz="0 0 0.0575" />
+        </joint>
+        <link name="pan_link">
+            <collision>
+                <origin rpy="0 0 0" xyz="0 0 0" />
+                <geometry>
+                    <mesh filename="file://$(find robot_arm_description)/urdf/meshes/pan_link.stl" scale="0.001 0.001 0.001" />
+                </geometry>
+            </collision>
+            <visual>
+                <origin rpy="0 0 0" xyz="0 0 0" />
+                <geometry>
+                    <mesh filename="file://$(find robot_arm_description)/urdf/meshes/pan_link.stl" scale="0.001 0.001 0.001" />
+                </geometry>
+                <material name="black" />
+            </visual>
+            <inertial>
+                <mass value="0.1" />
+                <inertia ixx="0.03" iyy="0.03" izz="0.03" ixy="0.0" ixz="0.0" iyz="0.0" />
+            </inertial>
+        </link>
+        <gazebo reference="pan_link">
+            <material>Gazebo/FlatBlack</material>
+        </gazebo>
+        <joint name="pan_joint" type="revolute">
+            <axis xyz="0 0 1" />
+            <limit effort="25" lower="-3.14159265359" upper="3.14159265359" velocity="1.5" />
+            <parent link="box_link" />
+            <child link="pan_link" />
+            <origin rpy="0 0 0" xyz="-0.012 0 0.002" />
+        </joint>
+        <link name="shoulder_link">
+            <collision>
+                <origin rpy="0 0 0" xyz="0 0 0" />
+                <geometry>
+                    <mesh filename="file://$(find robot_arm_description)/urdf/meshes/shoulder_link.stl" scale="0.001 0.001 0.001" />
+                </geometry>
+            </collision>
+            <visual>
+                <origin rpy="0 0 0" xyz="0 0 0" />
+                <geometry>
+                    <mesh filename="file://$(find robot_arm_description)/urdf/meshes/shoulder_link.stl" scale="0.001 0.001 0.001" />
+                </geometry>
+                <material name="black" />
+            </visual>
+            <inertial>
+                <mass value="0.1" />
+                <inertia ixx="0.03" iyy="0.03" izz="0.03" ixy="0.0" ixz="0.0" iyz="0.0" />
+            </inertial>
+        </link>
+        <gazebo reference="shoulder_link">
+            <material>Gazebo/FlatBlack</material>
+        </gazebo>
+        <joint name="shoulder_joint" type="revolute">
+            <axis xyz="0 1 0" />
+            <limit effort="25" lower="-1.8515" upper="2.1015" velocity="1.5" />
+            <parent link="pan_link" />
+            <child link="shoulder_link" />
+            <origin rpy="0 0 0" xyz="0 0 0.053" />
+        </joint>
+        <link name="elbow_link">
+            <collision>
+                <origin rpy="0 0 0" xyz="0 0 0" />
+                <geometry>
+                    <mesh filename="file://$(find robot_arm_description)/urdf/meshes/elbow_link.stl" scale="0.001 0.001 0.001" />
+                </geometry>
+            </collision>
+            <visual>
+                <origin rpy="0 0 0" xyz="0 0 0" />
+                <geometry>
+                    <mesh filename="file://$(find robot_arm_description)/urdf/meshes/elbow_link.stl" scale="0.001 0.001 0.001" />
+                </geometry>
+                <material name="black" />
+            </visual>
+            <inertial>
+                <mass value="0.1" />
+                <inertia ixx="0.03" iyy="0.03" izz="0.03" ixy="0.0" ixz="0.0" iyz="0.0" />
+            </inertial>
+        </link>
+        <gazebo reference="elbow_link">
+            <material>Gazebo/FlatBlack</material>
+        </gazebo>
+        <joint name="elbow_joint" type="revolute">
+            <axis xyz="0 1 0" />
+            <limit effort="25" lower="-0.4" upper="3.0" velocity="1.5" />
+            <parent link="shoulder_link" />
+            <child link="elbow_link" />
+            <origin rpy="0 0 0" xyz="0.03 0 0.2205" />
+        </joint>
+        <link name="wrist0_link">
+            <collision>
+                <origin rpy="0 0 0" xyz="0 0 0" />
+                <geometry>
+                    <mesh filename="file://$(find robot_arm_description)/urdf/meshes/wrist0_link.stl" scale="0.001 0.001 0.001" />
+                </geometry>
+            </collision>
+            <visual>
+                <origin rpy="0 0 0" xyz="0 0 0" />
+                <geometry>
+                    <mesh filename="file://$(find robot_arm_description)/urdf/meshes/wrist0_link.stl" scale="0.001 0.001 0.001" />
+                </geometry>
+                <material name="black" />
+            </visual>
+            <inertial>
+                <mass value="0.1" />
+                <inertia ixx="0.03" iyy="0.03" izz="0.03" ixy="0.0" ixz="0.0" iyz="0.0" />
+            </inertial>
+        </link>
+        <gazebo reference="wrist0_link">
+            <material>Gazebo/FlatBlack</material>
+        </gazebo>
+        <joint name="wrist0_joint" type="revolute">
+            <axis xyz="0 0 1" />
+            <limit effort="25" lower="-3.14159265359" upper="3.14159265359" velocity="1.5" />
+            <parent link="elbow_link" />
+            <child link="wrist0_link" />
+            <origin rpy="0 0 0" xyz="0.0 0 0.176" />
+        </joint>
+        <gazebo reference="wrist1_link">
+            <material>Gazebo/FlatBlack</material>
+        </gazebo>
+        <link name="wrist1_link">
+            <collision>
+                <origin rpy="0 0 0" xyz="0 0 0" />
+                <geometry>
+                    <mesh filename="file://$(find robot_arm_description)/urdf/meshes/wrist1_link.stl" scale="0.001 0.001 0.001" />
+                </geometry>
+            </collision>
+            <visual>
+                <origin rpy="0 0 0" xyz="0 0 0" />
+                <geometry>
+                    <mesh filename="file://$(find robot_arm_description)/urdf/meshes/wrist1_link.stl" scale="0.001 0.001 0.001" />
+                </geometry>
+                <material name="black" />
+            </visual>
+            <inertial>
+                <mass value="0.1" />
+                <inertia ixx="0.03" iyy="0.03" izz="0.03" ixy="0.0" ixz="0.0" iyz="0.0" />
+            </inertial>
+        </link>
+        <gazebo reference="wrist1_link">
+            <material>Gazebo/FlatBlack</material>
+        </gazebo>
+        <joint name="wrist1_joint" type="revolute">
+            <axis xyz="0 1 0" />
+            <limit effort="25" lower="-1.8" upper="2.0" velocity="1.5" />
+            <parent link="wrist0_link" />
+            <child link="wrist1_link" />
+            <origin rpy="0 0 0" xyz="0.0 0 0.0435" />
+        </joint>
+        <link name="wrist2_link" />
+        <joint name="wrist2_joint" type="revolute">
+            <axis xyz="0 0 1" />
+            <limit effort="25" lower="-3.14159265359" upper="3.14159265359" velocity="1.5" />
+            <parent link="wrist1_link" />
+            <child link="wrist2_link" />
+            <origin rpy="0 0 0" xyz="0.0 0 0.0715" />
+        </joint>
+        <link name="gripper_link">
+            <collision>
+                <origin rpy="0 0 0" xyz="0 0 0" />
+                <geometry>
+                    <mesh filename="file://$(find robot_arm_description)/urdf/meshes/gripper_link.stl" scale="0.001 0.001 0.001" />
+                </geometry>
+            </collision>
+            <visual>
+                <origin rpy="0 0 0" xyz="0 0 0" />
+                <geometry>
+                    <mesh filename="file://$(find robot_arm_description)/urdf/meshes/gripper_link.stl" scale="0.001 0.001 0.001" />
+                </geometry>
+                <material name="black" />
+            </visual>
+            <inertial>
+                <mass value="0.1" />
+                <inertia ixx="0.03" iyy="0.03" izz="0.03" ixy="0.0" ixz="0.0" iyz="0.0" />
+            </inertial>
+        </link>
+        <gazebo reference="gripper_link">
+            <material>Gazebo/FlatBlack</material>
+        </gazebo>
+        <joint name="gripper_joint" type="fixed">
+            <parent link="wrist2_link" />
+            <child link="gripper_link" />
+            <origin rpy="0 0 0" xyz="0.002784 0 0.1082" />
+        </joint>
+        <link name="finger_link">
+            <collision>
+                <origin rpy="0 0 0" xyz="0 0 0" />
+                <geometry>
+                    <mesh filename="file://$(find robot_arm_description)/urdf/meshes/finger_link.stl" scale="0.001 0.001 0.001" />
+                </geometry>
+            </collision>
+            <visual>
+                <origin rpy="0 0 0" xyz="0 0 0" />
+                <geometry>
+                    <mesh filename="file://$(find robot_arm_description)/urdf/meshes/finger_link.stl" scale="0.001 0.001 0.001" />
+                </geometry>
+                <material name="black" />
+            </visual>
+            <inertial>
+                <mass value="0.1" />
+                <inertia ixx="0.03" iyy="0.03" izz="0.03" ixy="0.0" ixz="0.0" iyz="0.0" />
+            </inertial>
+        </link>
+        <gazebo reference="finger_link">
+            <material>Gazebo/FlatBlack</material>
+        </gazebo>
+        <joint name="finger_joint" type="prismatic">
+            <axis xyz="0 1 0" />
+            <limit lower="0" upper="0.026" effort="1.0" velocity="0" />
+            <parent link="gripper_link" />
+            <child link="finger_link" />
             <origin rpy="0 0 0" xyz="0 0 0" />
-            <geometry>
-               <mesh filename="file://$(find robot_arm_description)/urdf/meshes/box_link.stl" scale="0.001 0.001 0.001" />
-            </geometry>
-         </collision>
-         <visual>
-            <origin rpy="0 0 0" xyz="0 0 0" />
-            <geometry>
-               <mesh filename="file://$(find robot_arm_description)/urdf/meshes/box_link.stl" scale="0.001 0.001 0.001" />
-            </geometry>
-            <material name="black" />
-         </visual>
-         <inertial>
-            <mass value="0.1" />
-            <inertia ixx="0.1" iyy="0.1" izz="0.1" ixy="0.0" ixz="0.0" iyz="0.0" />
-         </inertial>
-      </link>
-      <gazebo reference="box_link">
-         <material>Gazebo/FlatBlack</material>
-      </gazebo>
-      <joint name="base_to_mount" type="fixed">
-         <parent link="${parent}" />
-         <child link="box_link" />
-         <origin rpy="0 0 0" xyz="0 0 0.0575" />
-      </joint>
-      <link name="pan_link">
-         <collision>
-            <origin rpy="0 0 0" xyz="0 0 0" />
-            <geometry>
-               <mesh filename="file://$(find robot_arm_description)/urdf/meshes/pan_link.stl" scale="0.001 0.001 0.001" />
-            </geometry>
-         </collision>
-         <visual>
-            <origin rpy="0 0 0" xyz="0 0 0" />
-            <geometry>
-               <mesh filename="file://$(find robot_arm_description)/urdf/meshes/pan_link.stl" scale="0.001 0.001 0.001" />
-            </geometry>
-            <material name="black" />
-         </visual>
-         <inertial>
-            <mass value="0.1" />
-            <inertia ixx="0.03" iyy="0.03" izz="0.03" ixy="0.0" ixz="0.0" iyz="0.0" />
-         </inertial>
-      </link>
-      <gazebo reference="pan_link">
-         <material>Gazebo/FlatBlack</material>
-      </gazebo>
-      <joint name="pan_joint" type="revolute">
-         <axis xyz="0 0 1" />
-         <limit effort="25" lower="-3.14159265359" upper="3.14159265359" velocity="1.5" />
-         <parent link="box_link" />
-         <child link="pan_link" />
-         <origin rpy="0 0 0" xyz="-0.012 0 0.002" />
-      </joint>
-      <link name="shoulder_link">
-         <collision>
-            <origin rpy="0 0 0" xyz="0 0 0" />
-            <geometry>
-               <mesh filename="file://$(find robot_arm_description)/urdf/meshes/shoulder_link.stl" scale="0.001 0.001 0.001" />
-            </geometry>
-         </collision>
-         <visual>
-            <origin rpy="0 0 0" xyz="0 0 0" />
-            <geometry>
-               <mesh filename="file://$(find robot_arm_description)/urdf/meshes/shoulder_link.stl" scale="0.001 0.001 0.001" />
-            </geometry>
-            <material name="black" />
-         </visual>
-         <inertial>
-            <mass value="0.1" />
-            <inertia ixx="0.03" iyy="0.03" izz="0.03" ixy="0.0" ixz="0.0" iyz="0.0" />
-         </inertial>
-      </link>
-      <gazebo reference="shoulder_link">
-         <material>Gazebo/FlatBlack</material>
-      </gazebo>
-      <joint name="shoulder_joint" type="revolute">
-         <axis xyz="0 1 0" />
-         <limit effort="25" lower="-1.8515" upper="2.1015" velocity="1.5" />
-         <parent link="pan_link" />
-         <child link="shoulder_link" />
-         <origin rpy="0 0 0" xyz="0 0 0.053" />
-      </joint>
-      <link name="elbow_link">
-         <collision>
-            <origin rpy="0 0 0" xyz="0 0 0" />
-            <geometry>
-               <mesh filename="file://$(find robot_arm_description)/urdf/meshes/elbow_link.stl" scale="0.001 0.001 0.001" />
-            </geometry>
-         </collision>
-         <visual>
-            <origin rpy="0 0 0" xyz="0 0 0" />
-            <geometry>
-               <mesh filename="file://$(find robot_arm_description)/urdf/meshes/elbow_link.stl" scale="0.001 0.001 0.001" />
-            </geometry>
-            <material name="black" />
-         </visual>
-         <inertial>
-            <mass value="0.1" />
-            <inertia ixx="0.03" iyy="0.03" izz="0.03" ixy="0.0" ixz="0.0" iyz="0.0" />
-         </inertial>
-      </link>
-      <gazebo reference="elbow_link">
-         <material>Gazebo/FlatBlack</material>
-      </gazebo>
-      <joint name="elbow_joint" type="revolute">
-         <axis xyz="0 1 0" />
-         <limit effort="25" lower="-0.4" upper="3.0" velocity="1.5" />
-         <parent link="shoulder_link" />
-         <child link="elbow_link" />
-         <origin rpy="0 0 0" xyz="0.03 0 0.2205" />
-      </joint>
-      <link name="wrist0_link">
-         <collision>
-            <origin rpy="0 0 0" xyz="0 0 0" />
-            <geometry>
-               <mesh filename="file://$(find robot_arm_description)/urdf/meshes/wrist0_link.stl" scale="0.001 0.001 0.001" />
-            </geometry>
-         </collision>
-         <visual>
-            <origin rpy="0 0 0" xyz="0 0 0" />
-            <geometry>
-               <mesh filename="file://$(find robot_arm_description)/urdf/meshes/wrist0_link.stl" scale="0.001 0.001 0.001" />
-            </geometry>
-            <material name="black" />
-         </visual>
-         <inertial>
-            <mass value="0.1" />
-            <inertia ixx="0.03" iyy="0.03" izz="0.03" ixy="0.0" ixz="0.0" iyz="0.0" />
-         </inertial>
-      </link>
-      <gazebo reference="wrist0_link">
-         <material>Gazebo/FlatBlack</material>
-      </gazebo>
-      <joint name="wrist0_joint" type="revolute">
-         <axis xyz="0 0 1" />
-         <limit effort="25" lower="-3.14159265359" upper="3.14159265359" velocity="1.5" />
-         <parent link="elbow_link" />
-         <child link="wrist0_link" />
-         <origin rpy="0 0 0" xyz="0.0 0 0.176" />
-      </joint>
-      <gazebo reference="wrist1_link">
-         <material>Gazebo/FlatBlack</material>
-      </gazebo>
-      <link name="wrist1_link">
-         <collision>
-            <origin rpy="0 0 0" xyz="0 0 0" />
-            <geometry>
-               <mesh filename="file://$(find robot_arm_description)/urdf/meshes/wrist1_link.stl" scale="0.001 0.001 0.001" />
-            </geometry>
-         </collision>
-         <visual>
-            <origin rpy="0 0 0" xyz="0 0 0" />
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