Commit message: migrated to jazzy - harmonic stack

File: robot_arm_description/urdf/plugins.urdf.xacro (robot description, xacro)
@@ -4,10 +4,10 @@
       <xacro:if value="${gazebo}">
          <hardware>
-            <plugin>gazebo_ros2_control/GazeboSystem</plugin>
+            <plugin>gz_ros2_control/GazeboSimSystem</plugin>
          </hardware>
       </xacro:if>
       <xacro:unless value="${gazebo}">
          <hardware>
-            <plugin>fake_components/GenericSystem</plugin>
+            <plugin>mock_components/GenericSystem</plugin>
          </hardware>
       </xacro:unless>
@@ -21,5 +21,4 @@
          <param name="mimic">finger_joint</param>
          <param name="multiplier">1</param>
-         <command_interface name="position"/>
          <state_interface name="position" />
          <state_interface name="velocity" />
@@ -82,7 +81,5 @@
    </ros2_control>
    <gazebo>
-      <plugin filename="libgazebo_ros2_control.so" name="gazebo_ros2_control_urdf">
-         <robot_param>robot_description</robot_param>
-         <robot_param_node>robot_state_publisher</robot_param_node>
+      <plugin filename="gz_ros2_control-system" name="gz_ros2_control::GazeboSimROS2ControlPlugin">
          <parameters>$(find robot_arm_description)/config/controller.yaml</parameters>
       </plugin>

File: robot_arm_description/urdf/robot_arm.urdf.xacro (robot description, xacro)
@@ -28,13 +28,4 @@
          </inertial>
       </link>
-   <gazebo reference="base_mount">
-      <kp>1000000.0</kp>
-      <kd>1.0</kd>
-      <mu1>0.8</mu1>
-      <mu2>0.8</mu2>
-      <maxVel>0.0</maxVel>
-      <minDepth>0.001</minDepth>
-      <material>Gazebo/FlatBlack</material>
-   </gazebo>
-   <xacro:assembled_arm parent="base_mount" use_sim_time="$(arg use_sim_time)" />
+<xacro:assembled_arm parent="base_mount" use_sim_time="$(arg use_sim_time)" />
 </robot>
