Commit message: working gazebo simulation

File: robot_arm_description/urdf/arm_component.urdf.xacro (robot description, xacro)
@@ -54,4 +54,5 @@
             <child link="${child_frame_id}" />
             <origin rpy="0 0 0" xyz="${pos_x} ${pos_y} ${pos_z}" />
+            <dynamics damping="0.7" friction="100.0" />
         </joint>
     </xacro:macro>

File: robot_arm_description/urdf/arm_mech.urdf.xacro (robot description, xacro)
@@ -6,8 +6,8 @@
             frame_id="${parent}"
             child_frame_id="box_link"
-            mass="0.02"
+            mass="0.2"
             pos_x="0.0"
             pos_y="0.0"
-            pos_z="0.0575"
+            pos_z="0.0576"
             x_length="0.087"
             y_length="0.087"
@@ -28,5 +28,5 @@
             frame_id="box_link"
             child_frame_id="pan_link"
-            mass="0.0215"
+            mass="0.215"
             pos_x="-0.012"
             pos_y="0.0"
@@ -72,5 +72,5 @@
             frame_id="shoulder_link"
             child_frame_id="elbow_link"
-            mass="0.01"
+            mass="0.1"
             pos_x="0.03"
             pos_y="0.0"
@@ -94,5 +94,5 @@
             frame_id="elbow_link"
             child_frame_id="wrist0_link"
-            mass="0.01"
+            mass="0.1"
             pos_x="0.0"
             pos_y="0.0"
@@ -116,5 +116,5 @@
             frame_id="wrist0_link"
             child_frame_id="wrist1_link"
-            mass="0.01"
+            mass="0.1"
             pos_x="0.0"
             pos_y="0.0"
@@ -138,5 +138,5 @@
             frame_id="wrist1_link"
             child_frame_id="wrist2_link"
-            mass="0.01"
+            mass="0.1"
             pos_x="0.0"
             pos_y="0.0"

File: robot_arm_description/urdf/assembled_arm.urdf.xacro (robot description, xacro)
@@ -12,5 +12,5 @@
          <parent link="gripper_link" />
          <child link="tool_link" />
-         <origin rpy="0 -3.1416 0" xyz="0 0 -0.005" />
+         <origin rpy="0 -3.1416 0" xyz="0 0 0.1032" />
       </joint>
     </xacro:macro>

File: robot_arm_description/urdf/gripper_mech.urdf.xacro (robot description, xacro)
@@ -7,7 +7,7 @@
             child_frame_id="gripper_link"
             mass="0.01"
-            pos_x="0.002784"
+            pos_x="0.0"
             pos_y="0.0"
-            pos_z="0.1082"
+            pos_z="0.0"
             x_length="0.034"
             y_length="0.105"
@@ -29,7 +29,7 @@
             child_frame_id="finger_link"
             mass="0.01"
-            pos_x="0."
-            pos_y="0."
-            pos_z="0."
+            pos_x="0.002784"
+            pos_y="0.01408"
+            pos_z="0.0582"
             x_length="0.02"
             y_length="0.027"
@@ -51,7 +51,7 @@
             child_frame_id="mimic_finger_link"
             mass="0.01"
-            pos_x="0."
-            pos_y="0."
-            pos_z="0."
+            pos_x="0.002784"
+            pos_y="-0.01408"
+            pos_z="0.0582"
             x_length="0.02"
             y_length="0.027"

File: robot_arm_description/urdf/robot_arm.urdf.xacro (robot description, xacro)
@@ -22,11 +22,17 @@
       <inertial>
          <origin xyz="0 0 ${0.005/2.}" />
-         <mass value="10" />
-         <inertia ixx="${(1/12) * 10 * (0.09 * 0.09 + 0.005 * 0.005)}" ixy="0.0" ixz="0.0"
-            iyy="${(1/12) * 10 * (0.045 * 0.045 + 0.005 * 0.005)}" iyz="0.0"
-            izz="${(1/12) * 10 * (0.045 * 0.045 + 0.09 * 0.09)}" />
+         <mass value="3" />
+         <inertia ixx="${(1/12) * 10 * (0.15 * 0.15 + 0.005 * 0.005)}" ixy="0.0" ixz="0.0"
+            iyy="${(1/12) * 10 * (0.12 * 0.12 + 0.005 * 0.005)}" iyz="0.0"
+            izz="${(1/12) * 10 * (0.12 * 0.12 + 0.15 * 0.15)}" />
          </inertial>
       </link>
    <gazebo reference="base_mount">
+      <kp>1000000.0</kp>
+      <kd>1.0</kd>
+      <mu1>0.8</mu1>
+      <mu2>0.8</mu2>
+      <maxVel>0.0</maxVel>
+      <minDepth>0.001</minDepth>
       <material>Gazebo/FlatBlack</material>
    </gazebo>

Commit message: fixed rotation of joint for mimic joints

File: robot_arm_description/urdf/arm_component.urdf.xacro (robot description, xacro)
@@ -1,15 +1,10 @@
 <?xml version="1.0" encoding="UTF-8"?>
 <robot xmlns:xacro="http://ros.org/wiki/xacro">
-    <xacro:macro name="arm_component" params="frame_id child_frame_id mass pos_x pos_y pos_z x_length y_length z_length mesh mirror_mesh joint_name joint_type joint_axis joint_min joint_max joint_velocity joint_effort joint_to_mimic joint_mimic_multiplier">
-        <xacro:if value="${mirror_mesh}">
-            <xacro:property name="mesh_yaw" value="3.1416" />
-        </xacro:if>
-        <xacro:unless value="${mirror_mesh}">
-            <xacro:property name="mesh_yaw" value="0" />
-        </xacro:unless>
+    <xacro:macro name="arm_component" params="frame_id child_frame_id mass pos_x pos_y pos_z x_length y_length z_length mesh joint_name joint_type joint_axis joint_min joint_max joint_velocity joint_effort joint_to_mimic joint_mimic_multiplier">
+        <xacro:property name="joint_yaw" value="0" />
         <link name="${child_frame_id}">
             <xacro:if value="${mesh != ''}">
                 <collision>
-                    <origin rpy="0 0 ${mesh_yaw}" xyz="0 0 0" />
+                    <origin rpy="0 0 0" xyz="0 0 0" />
                     <geometry>
                         <mesh filename="${mesh}" scale="0.001 0.001 0.001" />
@@ -17,5 +12,5 @@
                 </collision>
                 <visual>
-                    <origin rpy="0 0 ${mesh_yaw}" xyz="0 0 0" />
+                    <origin rpy="0 0 0" xyz="0 0 0" />
                     <geometry>
                         <mesh filename="${mesh}" scale="0.001 0.001 0.001" />
@@ -47,4 +42,5 @@
                 </xacro:if>
                 <xacro:if value="${joint_to_mimic != ''}">
+                    <xacro:property name="joint_yaw" value="3.1416" />
                     <mimic joint="${joint_to_mimic}" multiplier="${joint_mimic_multiplier}" />
                 </xacro:if>
@@ -53,5 +49,5 @@
             <parent link="${frame_id}" />
             <child link="${child_frame_id}" />
-            <origin rpy="0 0 0" xyz="${pos_x} ${pos_y} ${pos_z}" />
+            <origin rpy="0 0 ${joint_yaw}" xyz="${pos_x} ${pos_y} ${pos_z}" />
             <dynamics damping="0.7" friction="100.0" />
         </joint>

File: robot_arm_description/urdf/arm_mech.urdf.xacro (robot description, xacro)
@@ -14,5 +14,4 @@
             z_length="0.04"
             mesh="file://$(find robot_arm_description)/urdf/meshes/box_link.stl"
-            mirror_mesh="false"
             joint_name="base_to_mount"
             joint_type="fixed"
@@ -36,5 +35,4 @@
             z_length="0.067"
             mesh="file://$(find robot_arm_description)/urdf/meshes/pan_link.stl"
-            mirror_mesh="false"
             joint_name="pan_joint"
             joint_type="revolute"
@@ -58,5 +56,4 @@
             z_length=".234"
             mesh="file://$(find robot_arm_description)/urdf/meshes/shoulder_link.stl"
-            mirror_mesh="false"
             joint_name="shoulder_joint"
             joint_type="revolute"
@@ -80,5 +77,4 @@
             z_length="0.168"
             mesh="file://$(find robot_arm_description)/urdf/meshes/elbow_link.stl"
-            mirror_mesh="false"
             joint_name="elbow_joint"
             joint_type="revolute"
@@ -102,5 +98,4 @@
             z_length="0.0547"
             mesh="file://$(find robot_arm_description)/urdf/meshes/wrist0_link.stl"
-            mirror_mesh="false"
             joint_name="wrist0_joint"
             joint_type="revolute"
@@ -124,5 +119,4 @@
             z_length="0.044"
             mesh="file://$(find robot_arm_description)/urdf/meshes/wrist1_link.stl"
-            mirror_mesh="false"
             joint_name="wrist1_joint"
             joint_type="revolute"
@@ -146,5 +140,4 @@
             z_length=""
             mesh=""
-            mirror_mesh="false"
             joint_name="wrist2_joint"
             joint_type="revolute"

File: robot_arm_description/urdf/gripper_mech.urdf.xacro (robot description, xacro)
@@ -14,5 +14,4 @@
             z_length="0.049"
             mesh="file://$(find robot_arm_description)/urdf/meshes/gripper_link.stl"
-            mirror_mesh="false"
             joint_name="gripper_joint"
             joint_type="fixed"
@@ -36,5 +35,4 @@
             z_length="0.05"
             mesh="file://$(find robot_arm_description)/urdf/meshes/finger_link.stl"
-            mirror_mesh="false"
             joint_name="finger_joint"
             joint_type="prismatic"
@@ -58,5 +56,4 @@
             z_length="0.05"
             mesh="file://$(find robot_arm_description)/urdf/meshes/finger_link.stl"
-            mirror_mesh="true"
             joint_name="mimic_finger_joint"
             joint_type="prismatic"
@@ -67,5 +64,5 @@
             joint_effort="1.0"
             joint_to_mimic="finger_joint"
-            joint_mimic_multiplier="-1"
+            joint_mimic_multiplier="1"
         />
     </xacro:macro>

File: robot_arm_description/urdf/plugins.urdf.xacro (robot description, xacro)
@@ -12,11 +12,14 @@
          </hardware>
       </xacro:unless>
+      <joint name="finger_joint">
+         <command_interface name="position"/>
+         <state_interface name="position" />
+         <state_interface name="velocity" />
+         <state_interface name="effort" />
+      </joint>
       <joint name="mimic_finger_joint">
          <param name="mimic">finger_joint</param>
-         <param name="multiplier">-1</param>
-         <command_interface name="position">
-            <param name="min">0</param>
-            <param name="max">0.026</param>
-         </command_interface>
+         <param name="multiplier">1</param>
+         <command_interface name="position"/>
          <state_interface name="position" />
          <state_interface name="velocity" />
@@ -77,13 +80,4 @@
          <state_interface name="effort" />
       </joint>
-      <joint name="finger_joint">
-         <command_interface name="position">
-            <param name="min">-3.1416</param>
-            <param name="max">3.1416</param>
-         </command_interface>
-         <state_interface name="position" />
-         <state_interface name="velocity" />
-         <state_interface name="effort" />
-      </joint>
    </ros2_control>
    <gazebo>

Commit message: fixed friction bug of each joints

File: robot_arm_description/urdf/arm_component.urdf.xacro (robot description, xacro)
@@ -27,7 +27,4 @@
             </xacro:if>
         </link>
-        <gazebo reference="${child_frame_id}">
-            <material>Gazebo/FlatBlack</material>
-        </gazebo>
         <joint name="${joint_name}" type="${joint_type}">
             <xacro:if value="${joint_type == 'revolute' or joint_type == 'prismatic'}">
@@ -50,5 +47,5 @@
             <child link="${child_frame_id}" />
             <origin rpy="0 0 ${joint_yaw}" xyz="${pos_x} ${pos_y} ${pos_z}" />
-            <dynamics damping="0.7" friction="100.0" />
+            <dynamics damping="0.7" friction="0.0" />
         </joint>
     </xacro:macro>

Commit message: fixed mimic joint error

File: robot_arm_description/urdf/arm_component.urdf.xacro (robot description, xacro)
@@ -40,5 +40,7 @@
                 <xacro:if value="${joint_to_mimic != ''}">
                     <xacro:property name="joint_yaw" value="3.1416" />
-                    <mimic joint="${joint_to_mimic}" multiplier="${joint_mimic_multiplier}" />
+                    <xacro:unless value="${gazebo}">
+                        <mimic joint="${joint_to_mimic}" multiplier="${joint_mimic_multiplier}" />
+                    </xacro:unless>
                 </xacro:if>
                 <limit effort="${joint_effort}" lower="${joint_min}" upper="${joint_max}" velocity="${joint_velocity}" />
